Commit message: orientation fixed

File: 2FG7_inwards_description/urdf/2FG7_inwards.xacro (robot description, xacro)
@@ -6,5 +6,5 @@
 <link name="base_link">
   <inertial>
-    <origin xyz="0.011012174829169266 0.02949692580937681 0.055310823797750784" rpy="0 0 0"/>
+    <origin xyz="-4.8989159583623376e-05 2.847569602502098e-06 0.06811082379775064" rpy="0 0 0"/>
     <mass value="1.2646523179240972"/>
     <inertia ixx="0.001504" iyy="0.001812" izz="0.001053" ixy="-0.0" iyz="0.0" ixz="-3e-06"/>
@@ -26,10 +26,10 @@
 <link name="right_finger_v1_1">
   <inertial>
-    <origin xyz="0.01878686731087252 3.0377198621395207e-06 0.02803421548623221" rpy="0 0 0"/>
+    <origin xyz="0.029847703322119633 0.029496959480087837 0.015234215486232036" rpy="0 0 0"/>
     <mass value="0.023219383355922288"/>
     <inertia ixx="6e-06" iyy="5e-06" izz="2e-06" ixy="-0.0" iyz="0.0" ixz="-1e-06"/>
   </inertial>
   <visual>
-    <origin xyz="0.032239 -0.029494 -0.09445" rpy="0 0 0"/>
+    <origin xyz="0.054361 0.029494 -0.12005" rpy="0 0 0"/>
     <geometry>
       <mesh filename="package://2FG7_inwards_description/meshes/right_finger_v1_1.stl" scale="0.001 0.001 0.001"/>
@@ -38,5 +38,5 @@
   </visual>
   <collision>
-    <origin xyz="0.032239 -0.029494 -0.09445" rpy="0 0 0"/>
+    <origin xyz="0.054361 0.029494 -0.12005" rpy="0 0 0"/>
     <geometry>
       <mesh filename="package://2FG7_inwards_description/meshes/right_finger_v1_1.stl" scale="0.001 0.001 0.001"/>
@@ -46,10 +46,10 @@
 <link name="left_finger_v1_1">
   <inertial>
-    <origin xyz="-0.018786539333398813 -2.881240314580452e-06 0.02803421548623866" rpy="0 0 0"/>
+    <origin xyz="-0.007725703322151688 0.029491040519911117 0.015234215486238503" rpy="0 0 0"/>
     <mass value="0.023219383355922288"/>
     <inertia ixx="6e-06" iyy="5e-06" izz="2e-06" ixy="-0.0" iyz="-0.0" ixz="1e-06"/>
   </inertial>
   <visual>
-    <origin xyz="-0.054361 -0.029494 -0.09445" rpy="0 0 0"/>
+    <origin xyz="-0.032239 0.029494 -0.12005" rpy="0 0 0"/>
     <geometry>
       <mesh filename="package://2FG7_inwards_description/meshes/left_finger_v1_1.stl" scale="0.001 0.001 0.001"/>
@@ -58,5 +58,5 @@
   </visual>
   <collision>
-    <origin xyz="-0.054361 -0.029494 -0.09445" rpy="0 0 0"/>
+    <origin xyz="-0.032239 0.029494 -0.12005" rpy="0 0 0"/>
     <geometry>
       <mesh filename="package://2FG7_inwards_description/meshes/left_finger_v1_1.stl" scale="0.001 0.001 0.001"/>
@@ -65,10 +65,10 @@
 </link>
 <joint name="right_finger_joint" type="fixed">
-  <origin xyz="-0.032239 0.029494 0.09445" rpy="0 0 0"/>
+  <origin xyz="-0.054361 -0.029494 0.12005" rpy="0 0 0"/>
   <parent link="base_link"/>
   <child link="right_finger_v1_1"/>
 </joint>
 <joint name="lef_finger_joint" type="prismatic">
-  <origin xyz="0.054361 0.029494 0.09445" rpy="0 0 0"/>
+  <origin xyz="0.032239 -0.029494 0.12005" rpy="0 0 0"/>
   <parent link="base_link"/>
   <child link="left_finger_v1_1"/>

File: 2FG7_outwards_description/urdf/2FG7_outwards.xacro (robot description, xacro)
@@ -6,6 +6,6 @@
 <link name="base_link">
   <inertial>
-    <origin xyz="0.011012174829169254 0.029496925809376805 0.05531082379775077" rpy="0 0 0"/>
-    <mass value="1.2646523179240974"/>
+    <origin xyz="-4.898915958379213e-05 2.84756960271082e-06 0.06811082379774974" rpy="0 0 0"/>
+    <mass value="1.2646523179240972"/>
     <inertia ixx="0.001504" iyy="0.001812" izz="0.001053" ixy="-0.0" iyz="0.0" ixz="-3e-06"/>
   </inertial>
@@ -26,10 +26,10 @@
 <link name="right_finger_v1_1">
   <inertial>
-    <origin xyz="0.006813460666601066 -2.8812403068227688e-06 0.0280342154862306" rpy="0 0 0"/>
+    <origin xyz="0.017874296677847158 0.02949104051991925 0.01523421548622829" rpy="0 0 0"/>
     <mass value="0.023219383355922288"/>
     <inertia ixx="6e-06" iyy="5e-06" izz="2e-06" ixy="-0.0" iyz="-0.0" ixz="1e-06"/>
   </inertial>
   <visual>
-    <origin xyz="0.032239 -0.029494 -0.09445" rpy="0 0 0"/>
+    <origin xyz="0.054361 0.029494 -0.12005" rpy="0 0 0"/>
     <geometry>
       <mesh filename="package://2FG7_outwards_description/meshes/right_finger_v1_1.stl" scale="0.001 0.001 0.001"/>
@@ -38,5 +38,5 @@
   </visual>
   <collision>
-    <origin xyz="0.032239 -0.029494 -0.09445" rpy="0 0 0"/>
+    <origin xyz="0.054361 0.029494 -0.12005" rpy="0 0 0"/>
     <geometry>
       <mesh filename="package://2FG7_outwards_description/meshes/right_finger_v1_1.stl" scale="0.001 0.001 0.001"/>
@@ -46,10 +46,10 @@
 <link name="left_finger_v1_1">
   <inertial>
-    <origin xyz="-0.006813132689127449 3.0377198543818373e-06 0.028034215486240202" rpy="0 0 0"/>
+    <origin xyz="0.004247703322119739 0.029496959480080673 0.015234215486237948" rpy="0 0 0"/>
     <mass value="0.023219383355922288"/>
     <inertia ixx="6e-06" iyy="5e-06" izz="2e-06" ixy="-0.0" iyz="0.0" ixz="-1e-06"/>
   </inertial>
   <visual>
-    <origin xyz="-0.054361 -0.029494 -0.09445" rpy="0 0 0"/>
+    <origin xyz="-0.032239 0.029494 -0.12005" rpy="0 0 0"/>
     <geometry>
       <mesh filename="package://2FG7_outwards_description/meshes/left_finger_v1_1.stl" scale="0.001 0.001 0.001"/>
@@ -58,5 +58,5 @@
   </visual>
   <collision>
-    <origin xyz="-0.054361 -0.029494 -0.09445" rpy="0 0 0"/>
+    <origin xyz="-0.032239 0.029494 -0.12005" rpy="0 0 0"/>
     <geometry>
       <mesh filename="package://2FG7_outwards_description/meshes/left_finger_v1_1.stl" scale="0.001 0.001 0.001"/>
@@ -65,10 +65,10 @@
 </link>
 <joint name="right_finger_joint" type="fixed">
-  <origin xyz="-0.032239 0.029494 0.09445" rpy="0 0 0"/>
+  <origin xyz="-0.054361 -0.029494 0.12005" rpy="0 0 0"/>
   <parent link="base_link"/>
   <child link="right_finger_v1_1"/>
 </joint>
 <joint name="lef_finger_joint" type="prismatic">
-  <origin xyz="0.054361 0.029494 0.09445" rpy="0 0 0"/>
+  <origin xyz="0.032239 -0.029494 0.12005" rpy="0 0 0"/>
   <parent link="base_link"/>
   <child link="left_finger_v1_1"/>
