Commit message: link name changed

File: 2FG7_outwards_description/urdf/2FG7_outwards.trans.xacro (robot description, xacro)
@@ -14,25 +14,2 @@
   </xacro:macro>
 </robot>
- <!--
-<robot name="2FG7_outwards" xmlns:xacro="http://www.ros.org/wiki/xacro" >
-<transmission name="left_finger_joint_tran">
-  <type>transmission_interface/SimpleTransmission</type>
-    <joint name="left_finger_joint">
-      <hardwareInterface>hardware_interface/PositionJointInterface</hardwareInterface>
-    </joint>
-  <actuator name="left_finger_joint_motor">
-    <hardwareInterface>hardware_interface/PositionJointInterface</hardwareInterface>
-    <mechanicalReduction>1</mechanicalReduction>
-  </actuator>
-</transmission>
-<! <transmission name="right_finger_joint_tran">
-  <type>transmission_interface/SimpleTransmission</type>
-    <joint name="right_finger_joint">
-      <hardwareInterface>hardware_interface/PositionJointInterface</hardwareInterface>
-    </joint>
-  <actuator name="right_finger_joint_motor">
-    <hardwareInterface>hardware_interface/PositionJointInterface</hardwareInterface>
-    <mechanicalReduction>1</mechanicalReduction>
-  </actuator>
-</transmission>
-</robot>  -->

File: 2FG7_outwards_description/urdf/2FG7_outwards.xacro (robot description, xacro)
@@ -1,7 +1,7 @@
 <?xml version="1.0" ?>
 <robot name="2FG7_outwards" xmlns:xacro="http://www.ros.org/wiki/xacro">
-<xacro:include filename="$(find 2FG7_outwards_description)/urdf/materials.xacro" />
-<xacro:include filename="$(find 2FG7_outwards_description)/urdf/2FG7_outwards.trans.xacro" />
-<xacro:include filename="$(find 2FG7_outwards_description)/urdf/2FG7_outwards.gazebo" />
+<xacro:include filename="$(find onrobot_2fg7_description)/urdf/materials.xacro" />
+<xacro:include filename="$(find onrobot_2fg7_description)/urdf/2FG7_outwards.trans.xacro" />
+<xacro:include filename="$(find onrobot_2fg7_description)/urdf/2FG7_outwards.gazebo" />
 <xacro:gripper_transmission/>
 <link name="gripper_base_link">
@@ -14,5 +14,5 @@
     <origin xyz="0 0 0" rpy="0 0 0"/>
     <geometry>
-      <mesh filename="package://2FG7_outwards_description/meshes/base_link.stl" scale="0.001 0.001 0.001"/>
+      <mesh filename="package://onrobot_2fg7_description/meshes/base_link.stl" scale="0.001 0.001 0.001"/>
     </geometry>
     <material name="silver"/>
@@ -21,9 +21,9 @@
     <origin xyz="0 0 0" rpy="0 0 0"/>
     <geometry>
-      <mesh filename="package://2FG7_outwards_description/meshes/base_link.stl" scale="0.001 0.001 0.001"/>
+      <mesh filename="package://onrobot_2fg7_description/meshes/base_link.stl" scale="0.001 0.001 0.001"/>
     </geometry>
   </collision>
 </link>
-<link name="right_finger_v1_1">
+<link name="right_finger_link">
   <inertial>
     <origin xyz="0.017874296677847158 0.02949104051991925 0.01523421548622829" rpy="0 0 0"/>
@@ -34,5 +34,5 @@
     <origin xyz="0.054361 0.029494 -0.12005" rpy="0 0 0"/>
     <geometry>
-      <mesh filename="package://2FG7_outwards_description/meshes/right_finger_v1_1.stl" scale="0.001 0.001 0.001"/>
+      <mesh filename="package://onrobot_2fg7_description/meshes/right_finger_link.stl" scale="0.001 0.001 0.001"/>
     </geometry>
     <material name="silver"/>
@@ -41,9 +41,9 @@
     <origin xyz="0.054361 0.029494 -0.12005" rpy="0 0 0"/>
     <geometry>
-      <mesh filename="package://2FG7_outwards_description/meshes/right_finger_v1_1.stl" scale="0.001 0.001 0.001"/>
+      <mesh filename="package://onrobot_2fg7_description/meshes/right_finger_link.stl" scale="0.001 0.001 0.001"/>
     </geometry>
   </collision>
 </link>
-<link name="left_finger_v1_1">
+<link name="left_finger_link">
   <inertial>
     <origin xyz="0.004247703322119739 0.029496959480080673 0.015234215486237948" rpy="0 0 0"/>
@@ -54,5 +54,5 @@
     <origin xyz="-0.032239 0.029494 -0.12005" rpy="0 0 0"/>
     <geometry>
-      <mesh filename="package://2FG7_outwards_description/meshes/left_finger_v1_1.stl" scale="0.001 0.001 0.001"/>
+      <mesh filename="package://onrobot_2fg7_description/meshes/left_finger_link.stl" scale="0.001 0.001 0.001"/>
     </geometry>
     <material name="silver"/>
@@ -61,5 +61,5 @@
     <origin xyz="-0.032239 0.029494 -0.12005" rpy="0 0 0"/>
     <geometry>
-      <mesh filename="package://2FG7_outwards_description/meshes/left_finger_v1_1.stl" scale="0.001 0.001 0.001"/>
+      <mesh filename="package://onrobot_2fg7_description/meshes/left_finger_link.stl" scale="0.001 0.001 0.001"/>
     </geometry>
   </collision>
@@ -68,5 +68,5 @@
   <origin xyz="0.032239 -0.029494 0.12005" rpy="0 0 0"/>
   <parent link="gripper_base_link"/>
-  <child link="left_finger_v1_1"/>
+  <child link="left_finger_link"/>
   <axis xyz="-1.0 0.0 0.0"/>
   <limit lower="0.0" upper="0.019" effort="140" velocity="0.45"/> <!-- total 0.38 -->
@@ -75,5 +75,5 @@
   <origin xyz="-0.054361 -0.029494 0.12005" rpy="0 0 0"/>
   <parent link="gripper_base_link"/>
-  <child link="right_finger_v1_1"/>
+  <child link="right_finger_link"/>
   <axis xyz="1.0 0.0 0.0"/>
   <limit lower="-0.019" upper="0.019" effort="140" velocity="0.45"/>

File: 2FG7_outwards_description/urdf/2FG7_outwards_upload.xacro (robot description, xacro)
@@ -1,5 +1,5 @@
 <?xml version="1.0" ?>
 <robot name="2FG7_outwards" xmlns:xacro="http://www.ros.org/wiki/xacro">
-  <xacro:include filename="$(find 2FG7_outwards_description)/urdf/2FG7_outwards.xacro" />
+  <xacro:include filename="$(find onrobot_2fg7_description)/urdf/2FG7_outwards.xacro" />
   <link name="world" />
   <joint name="world_joint" type="fixed">
@@ -8,6 +8,6 @@
     <origin xyz="0.0 0.0 0.0" rpy="0.0 0.0 0.0" />
   </joint>
-  <xacro:include filename="$(find 2FG7_outwards_description)/urdf/gzplugin_grasp_fix.urdf.xacro"/>
-  <xacro:include filename="$(find 2FG7_outwards_description)/urdf/mimic_fix.urdf.xacro"/>
+  <xacro:include filename="$(find onrobot_2fg7_description)/urdf/gzplugin_grasp_fix.urdf.xacro"/>
+  <xacro:include filename="$(find onrobot_2fg7_description)/urdf/mimic_fix.urdf.xacro"/>
   <xacro:gzplugin_grasp_fix/>
   <xacro:mimic_fix/>

File: 2FG7_outwards_description/urdf/gzplugin_grasp_fix.urdf.xacro (robot description, xacro)
@@ -8,6 +8,6 @@
 					<arm_name>2FG7</arm_name>
 					<palm_link>gripper_base_link</palm_link>
-					<gripper_link>left_finger_v1_1</gripper_link>
-					<gripper_link>right_finger_v1_1</gripper_link>
+					<gripper_link>left_finger_link</gripper_link>
+					<gripper_link>right_finger_link</gripper_link>
 				</arm>
 				<forces_angle_tolerance>80</forces_angle_tolerance>
