Commit message: inwards config added

File: urdf/gzplugin_grasp_fix.urdf.xacro (robot description, xacro)
@@ -7,5 +7,5 @@
 				<arm>
 					<arm_name>2FG7</arm_name>
-					<palm_link>gripper_base_link</palm_link>
+					<palm_link>base_link</palm_link>
 					<gripper_link>left_finger_link</gripper_link>
 					<gripper_link>right_finger_link</gripper_link>

File: urdf/onrobot_2fg7_upload.xacro (robot description, xacro)
@@ -1,9 +1,10 @@
 <?xml version="1.0" ?>
-<robot name="2FG7_outwards" xmlns:xacro="http://www.ros.org/wiki/xacro">
-  <xacro:include filename="$(find onrobot_2fg7_description)/urdf/2FG7_outwards.xacro" />
+<robot name="2fg7_outwards" xmlns:xacro="http://www.ros.org/wiki/xacro">
+  <xacro:include filename="$(find onrobot_2fg7_description)/urdf/onrobot_2fg7.xacro" />
+ <xacro:onrobot_2fg7_gripper prefix="" finger_configuration="outwards"/>
   <link name="world" />
   <joint name="world_joint" type="fixed">
     <parent link="world" />
-    <child link = "gripper_base_link" />
+    <child link = "base_link" />
     <origin xyz="0.0 0.0 0.0" rpy="0.0 0.0 0.0" />
   </joint>
